File: EagleCAD/iswitchpihat/iswitchpihat.brd (EAGLE design)
At the start: 65 x 56.5 mm, 35 parts, among them IC1 ATTINY24/44/84-PU, IC2 MIC2025-1YM

Commit message: small changes
Parts:
- moved S2 0.63 mm to (57.7, 41.8)
Routing:
- net N$16: track 66.1 -> 67.1 mm
- net N$6: track 43.5 -> 44.6 mm
- net N$20: track 14.8 -> 14.0 mm
Other:
- board text added: "iSwitchPi Ver. 3.1"
- board text removed: "iSwitchPi Ver. 3"
Changed lines of the file:
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@@
 <wire x1="65" y1="56.5" x2="0" y2="56.5" width="0" layer="20"/>
 <wire x1="0" y1="56.5" x2="0" y2="0" width="0" layer="20"/>
-<text x="21.59" y="13.97" size="1.524" layer="21">iSwitchPi Ver. 3</text>
+<text x="20.32" y="13.97" size="1.524" layer="21">iSwitchPi Ver. 3.1</text>
 <hole x="3.5" y="52.5" drill="3.2"/>
 <hole x="61.5" y="52.5" drill="2.8"/>
@@
 <attribute name="VALUE" x="55.88" y="4.445" size="0.762" layer="27" rot="R180"/>
 </element>
-<element name="S2" library="switch-dil" package="DIP04S" value="" x="57.1" y="41.83" smashed="yes">
-<attribute name="MF" value="" x="57.1" y="41.83" size="1.778" layer="27" display="off"/>
-<attribute name="OC_NEWARK" value="unknown" x="57.1" y="41.83" size="1.778" layer="27" display="off"/>
-<attribute name="MPN" value="" x="57.1" y="41.83" size="1.778" layer="27" display="off"/>
-<attribute name="OC_FARNELL" value="unknown" x="57.1" y="41.83" size="1.778" layer="27" display="off"/>
-<attribute name="NAME" x="49.48" y="45.386" size="1.016" layer="25" ratio="10"/>
-<attribute name="VALUE" x="57.608" y="46.656" size="1.27" layer="27" ratio="10"/>
+<element name="S2" library="switch-dil" package="DIP04S" value="" x="57.735" y="41.83" smashed="yes">
+<attribute name="MF" value="" x="57.735" y="41.83" size="1.778" layer="27" display="off"/>
+<attribute name="OC_NEWARK" value="unknown" x="57.735" y="41.83" size="1.778" layer="27" display="off"/>
+<attribute name="MPN" value="" x="57.735" y="41.83" size="1.778" layer="27" display="off"/>
+<attribute name="OC_FARNELL" value="unknown" x="57.735" y="41.83" size="1.778" layer="27" display="off"/>
+<attribute name="NAME" x="50.115" y="45.386" size="1.016" layer="25" ratio="10"/>
+<attribute name="VALUE" x="58.243" y="46.656" size="1.27" layer="27" ratio="10"/>
 </element>
 <element name="C1" library="rcl" package="C1206" value="1uF" x="19.05" y="31.75" smashed="yes" rot="R180">
@@
 <wire x1="27.94" y1="22.86" x2="27.81" y2="22.86" width="0.2" layer="1"/>
 <wire x1="53.34" y1="23.495" x2="53.67" y2="23.51" width="0.2" layer="16"/>
-<wire x1="18.415" y1="29.21" x2="17.78" y2="27.94" width="0.2" layer="1"/>
-<wire x1="24.765" y1="23.495" x2="18.415" y2="29.21" width="0.2" layer="16"/>
+<wire x1="18.415" y1="29.845" x2="17.78" y2="27.94" width="0.2" layer="1"/>
+<wire x1="24.765" y1="23.495" x2="18.415" y2="29.845" width="0.2" layer="16"/>
 <wire x1="26.035" y1="23.495" x2="24.765" y2="23.495" width="0.2" layer="16"/>
 <wire x1="26.67" y1="23.495" x2="26.035" y2="23.495" width="0.2" layer="1"/>
@@
 <wire x1="27.305" y1="22.86" x2="27.81" y2="22.86" width="0.2" layer="1"/>
 <via x="48.26" y="23.495" extent="1-16" drill="0.35"/>
-<via x="18.415" y="29.21" extent="1-16" drill="0.35"/>
+<via x="18.415" y="29.845" extent="1-16" drill="0.35"/>
 <via x="26.035" y="23.495" extent="1-16" drill="0.35"/>
 </signal>
@@
 <wire x1="62.23" y1="32.385" x2="62.865" y2="31.75" width="0.2" layer="1"/>
 <wire x1="60.325" y1="32.385" x2="62.23" y2="32.385" width="0.2" layer="1"/>
-<wire x1="55.245" y1="37.465" x2="60.325" y2="32.385" width="0.2" layer="1"/>
+<wire x1="56.515" y1="36.195" x2="60.325" y2="32.385" width="0.2" layer="1"/>
 <wire x1="61.595" y1="28.575" x2="61.29" y2="28.59" width="0.2" layer="1"/>
-<wire x1="55.245" y1="37.465" x2="55.83" y2="38.02" width="0.2" layer="1"/>
+<wire x1="56.515" y1="36.195" x2="56.465" y2="38.02" width="0.2" layer="1"/>
 </signal>
 <signal name="N$21">
@@
 <wire x1="60.96" y1="36.195" x2="63.5" y2="33.655" width="0.2" layer="1"/>
 <wire x1="59.69" y1="36.195" x2="60.96" y2="36.195" width="0.2" layer="1"/>
-<wire x1="58.42" y1="37.465" x2="59.69" y2="36.195" width="0.2" layer="1"/>
+<wire x1="59.055" y1="36.195" x2="59.69" y2="36.195" width="0.2" layer="1"/>
 <wire x1="61.595" y1="23.495" x2="61.29" y2="23.51" width="0.2" layer="1"/>
-<wire x1="58.42" y1="37.465" x2="58.37" y2="38.02" width="0.2" layer="1"/>
+<wire x1="59.055" y1="36.195" x2="59.005" y2="38.02" width="0.2" layer="1"/>
 </signal>
 <signal name="N$18">
@@
 <wire x1="64.135" y1="23.495" x2="61.595" y2="20.955" width="0.2" layer="1"/>
 <wire x1="64.135" y1="34.29" x2="64.135" y2="23.495" width="0.2" layer="1"/>
-<wire x1="60.96" y1="37.465" x2="64.135" y2="34.29" width="0.2" layer="1"/>
+<wire x1="62.23" y1="37.465" x2="64.135" y2="34.29" width="0.2" layer="1"/>
 <wire x1="61.595" y1="20.955" x2="61.29" y2="20.97" width="0.2" layer="1"/>
-<wire x1="60.96" y1="37.465" x2="60.91" y2="38.02" width="0.2" layer="1"/>
+<wire x1="62.23" y1="37.465" x2="61.545" y2="38.02" width="0.2" layer="1"/>
 </signal>
 <signal name="N$11">
@@
 <contactref element="IC1" pad="6"/>
 <contactref element="S2" pad="1"/>
-<wire x1="59.69" y1="31.115" x2="53.34" y2="37.465" width="0.2" layer="1"/>
+<wire x1="59.69" y1="31.115" x2="54.61" y2="36.195" width="0.2" layer="1"/>
 <wire x1="60.96" y1="31.115" x2="59.69" y2="31.115" width="0.2" layer="1"/>
-<wire x1="53.34" y1="37.465" x2="53.29" y2="38.02" width="0.2" layer="1"/>
+<wire x1="54.61" y1="36.195" x2="53.925" y2="38.02" width="0.2" layer="1"/>
 <wire x1="60.96" y1="31.115" x2="61.29" y2="31.13" width="0.2" layer="1"/>
 </signal>
@@
 <wire x1="41.275" y1="43.815" x2="39.37" y2="45.72" width="0.2" layer="1"/>
 <wire x1="59.055" y1="43.815" x2="41.275" y2="43.815" width="0.2" layer="1"/>
-<wire x1="59.69" y1="44.45" x2="59.055" y2="43.815" width="0.2" layer="1"/>
-<wire x1="59.69" y1="53.975" x2="59.69" y2="44.45" width="0.2" layer="1"/>
-<wire x1="57.785" y1="55.88" x2="59.69" y2="53.975" width="0.2" layer="1"/>
-<wire x1="28.575" y1="55.88" x2="57.785" y2="55.88" width="0.2" layer="1"/>
+<wire x1="60.325" y1="44.45" x2="59.055" y2="43.815" width="0.2" layer="1"/>
+<wire x1="59.055" y1="53.975" x2="60.325" y2="44.45" width="0.2" layer="1"/>
+<wire x1="59.055" y1="55.88" x2="59.055" y2="53.975" width="0.2" layer="1"/>
+<wire x1="28.575" y1="55.88" x2="59.055" y2="55.88" width="0.2" layer="1"/>
 <wire x1="26.67" y1="53.975" x2="28.575" y2="55.88" width="0.2" layer="1"/>
 <wire x1="26.67" y1="53.975" x2="26.15" y2="53.77" width="0.2" layer="1"/>

Commit message: many thing updated for new board
Parts:
- removed J1, J2: (no value), SparkFun-Connectors:1X02
- removed JP2: (no value), adafruit:1X01
- removed R5: 320, resistor:0204/7
- removed RTRIM: 50k, iswitchpihat:TEST2TEST2_3362
- added S4: (no value), switch-dil:DIP04S
- added TESTPINS: (no value), SparkFun-Connectors:1X02
- C4: value 100uF -> 1uF
- moved R7 7.73 mm to (54.6, 10.2), turned to 270 degrees
- moved R8 7.24 mm to (37.5, 28.6), turned to 270 degrees
- moved R2 5.12 mm to (45.7, 24.7), turned to 90 degrees
- moved R4 5.08 mm to (38.1, 10.2)
- moved R1 4.02 mm to (41.9, 28.9), turned to 270 degrees
- moved C4 3.81 mm to (19.1, 12.7)
- moved R3 3.81 mm to (19.1, 17.8)
- moved JP1 2.54 mm to (8.89, 16.5)
- moved JP5 1.42 mm to (22.9, 34.9)
- moved S1 1.42 mm to (31.8, 6.35), turned to 90 degrees
- moved LED1 1.27 mm to (41.9, 2.54)
- moved LED2 1.27 mm to (52.1, 2.54)
- moved R6 1.27 mm to (34.3, 26.7)
- moved JP4 0.63 mm to (21.0, 38.1)
- renumbered JP3 to GND
Connections:
- net 3.3V: no longer RTRIM.2
- net GND: now also S4.1, S4.2; no longer J2.1, R5.1
- net N$11: now also R7.1, S4.3; no longer IC1.7, RTRIM.3
- net N$14: now also R7.2; no longer R7.1
- net N$17: now also R4.2, S4.4; no longer R5.2, RTRIM.1
- net N$26: now also IC1.7, S4.7; no longer J1.1, R4.2
- net N$27: now also S4.8; no longer J2.2, JP1.8
- net N$28: now also S4.6, TESTPINS.1; no longer JP2.1, R7.2
- net N$8: now also TESTPINS.2
- net N$9: now also S4.5; no longer J1.2
Routing:
- net N$26: track 8.03 -> 41.1 mm
- net N$27: track 50.5 -> 18.0 mm, vias 1 -> 0
- net N$1: track 103.3 -> 73.5 mm
- net N$11: track 30.0 -> 9.62 mm
- net N$9: track 43.7 -> 63.9 mm
- net 3.3V: track 73.1 -> 57.7 mm
- net N$17: track 6.66 -> 18.9 mm
- net GND: track 49.4 -> 58.1 mm
- net N$21: track 18.6 -> 27.0 mm
- net N$8: track 12.7 -> 20.3 mm
- net N$14: track 9.57 -> 4.56 mm
- net N$6: track 44.6 -> 40.8 mm
- net N$16: track 67.1 -> 70.8 mm, vias 0 -> 1
- net N$28: track 48.5 -> 52.1 mm
- net N$7: track 22.1 -> 24.8 mm
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Other:
- board text added: "iSwitchPi Ver. 3.2"
- board text removed: "iSwitchPi Ver. 3.1"
