File: EagleCAD/iswitchpihat/iswitchpihat.sch (EAGLE design)
At the start: 35 parts, among them IC1 ATTINY24/44/84-PU, IC2 MIC2025-1YM

Commit message: many thing updated for new board
Parts:
- removed J1, J2: (no value), SparkFun-Connectors:M02PTH
- removed JP2: (no value), adafruit:PINHD-1X1
- removed R5: 320, resistor:R-EU_0204/7
- removed RTRIM: 50k, iswitchpihat:R-TRIMM3362
- added S4: (no value), switch-dil:DIP04S
- added TESTPINS: (no value), SparkFun-Connectors:M02PTH
- C4: value 100uF -> 1uF
- renumbered JP3 to GND
Connections:
- net 3.3V: no longer RTRIM.C
- net GND: now also S4-1.1, S4-2.1; no longer J2.1, R5.1
- net N$11: now also R7.1, S4-3.1; no longer IC1.(PCINT6/OC1A/SDA/MOSI/ADC6)PA6, RTRIM.B
- net N$14: now also R7.2; no longer R7.1
- net N$17: now also R4.2, S4-4.1; no longer R5.2, RTRIM.A
- net N$26: now also IC1.(PCINT6/OC1A/SDA/MOSI/ADC6)PA6, S4-2.2; no longer J1.1, R4.2
- net N$27: now also S4-1.2; no longer J2.2, JP1.8
- net N$28: now also S4-3.2, TESTPINS.1; no longer JP2.1, R7.2
- net N$8: now also TESTPINS.2
- net N$9: now also S4-4.2; no longer J1.2
Other:
- note added: "Intelligent ON-OFF Switch for Raspberry Pi iSwitchPi Ver 2"
- note added: "R9 only needed if IC2 is MIC2445A"
- note added: "Test Pins"
- note added: "Testpin 5V"
- note added: "To be connected"
- note removed: "Intelligent ON-OFF Switch for Raspberry Pi iSwitchPi Ver 3"
- note removed: "Trim Frequency"
- moved on the sheet: JP5, JP6, LED1, LED2, R4, R6, R7
